File: SCAN2000_driver/SCAN2000_driver.kicad_pcb (KiCad board)
At the start: 2 copper layers, 40 x 53.3 mm, 24 parts, among them J1 IDC-Header_2x13, J2 Header 2x13, U1 74LVC541A, U2 74LVC541A, U3 74LVC541A

Commit message: better doc
Parts:
- U1, U2, U3: value 74LVC541A -> 74LVC541AP; footprint Package_SO:SO-20_12.8x7.5mm_P1.27mm -> Package_SO:TSSOP-20_4.4x6.5mm_P0.65mm
- moved U3 6.23 mm to (95.4, 79.6)
- moved C2 5.88 mm to (97.8, 48.8), turned to 0 degrees
- moved F1 5.71 mm to (86.6, 89.4)
- moved C1 5.63 mm to (97.6, 50.5)
- moved C6 5.54 mm to (97.8, 73.5), turned to 0 degrees
- moved J2 5.33 mm to (84.1, 54.6)
- moved C4 5.00 mm to (97.9, 62.6), turned to 0 degrees
- moved U1 4.49 mm to (95.4, 54.9)
- moved U2 3.94 mm to (95.4, 68.7)
- moved C3 3.78 mm to (97.7, 64.4)
- moved C5 1.57 mm to (97.6, 75.3)
Routing:
- net +3.3V: track 100.2 -> 69.3 mm
- net GND: track 22.8 -> 37.0 mm, vias 9 -> 17
- net /P22: track 13.4 -> 7.06 mm
- net /P20: track 14.4 -> 8.40 mm
- net /P21: track 12.5 -> 6.64 mm
- net /P19: track 13.8 -> 8.18 mm
- net /P18: track 19.3 -> 14.2 mm
- net /P17: track 17.7 -> 13.2 mm
- net /P1: track 11.6 -> 7.35 mm
- net /P2: track 11.1 -> 7.23 mm
- net Net-(J2-Pin_22): track 9.83 -> 6.31 mm
- net /P3: track 10.9 -> 7.64 mm
- net /P5: track 11.7 -> 8.60 mm
- net Net-(J2-Pin_21): track 12.5 -> 9.38 mm
- net /P16: track 10.0 -> 6.96 mm
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Other:
- board size 40 x 53.3 mm -> 34.7 x 53.3 mm
- board text added: "Mezzanine board for SCAN2000, Driver/ESD protection V1.0"
- board text removed: "Mezzanine board for SCAN2000, driver V1.0"
