File: SCAN2000_driver/SCAN2000_driver.kicad_sch (KiCad schematic)
At the start: 24 parts, among them J2 Header 2x13, J21 IDC-Header_2x13, U1 74LVC541A, U2 74LVC541A, U3 74LVC541A

Commit message: better doc
Parts:
- U1, U2, U3: value 74LVC541A -> 74LVC541AP; footprint Package_SO:SO-20_12.8x7.5mm_P1.27mm -> Package_SO:TSSOP-20_4.4x6.5mm_P0.65mm
Changed lines of the file:
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@@
       (effects (font (size 1.27 1.27)) (justify left))
     )
-    (property "Value" "74LVC541A" (at 107.3659 134.8011 0)
-      (effects (font (size 1.27 1.27)) (justify left))
-    )
-    (property "Footprint" "Package_SO:SO-20_12.8x7.5mm_P1.27mm" (at 105.41 151.13 0)
+    (property "Value" "74LVC541AP" (at 107.3659 134.8011 0)
+      (effects (font (size 1.27 1.27)) (justify left))
+    )
+    (property "Footprint" "Package_SO:TSSOP-20_4.4x6.5mm_P0.65mm" (at 105.41 151.13 0)
       (effects (font (size 1.27 1.27)) hide)
     )
@@
       (effects (font (size 1.27 1.27)) (justify left))
     )
-    (property "Value" "74LVC541A" (at 107.3659 23.0411 0)
-      (effects (font (size 1.27 1.27)) (justify left))
-    )
-    (property "Footprint" "Package_SO:SO-20_12.8x7.5mm_P1.27mm" (at 105.41 39.37 0)
+    (property "Value" "74LVC541AP" (at 107.3659 23.0411 0)
+      (effects (font (size 1.27 1.27)) (justify left))
+    )
+    (property "Footprint" "Package_SO:TSSOP-20_4.4x6.5mm_P0.65mm" (at 105.41 39.37 0)
       (effects (font (size 1.27 1.27)) hide)
     )
@@
       (effects (font (size 1.27 1.27)) (justify left))
     )
-    (property "Value" "74LVC541A" (at 107.3659 78.9211 0)
-      (effects (font (size 1.27 1.27)) (justify left))
-    )
-    (property "Footprint" "Package_SO:SO-20_12.8x7.5mm_P1.27mm" (at 105.41 95.25 0)
-      (effects (font (size 1.27 1.27)) hide)
-    )
+    (property "Value" "74LVC541AP" (at 107.3659 78.9211 0)
+      (effects (font (size 1.27 1.27)) (justify left))
+    )
+    (property "Footprint" "Package_SO:TSSOP-20_4.4x6.5mm_P0.65mm" (at 105.41 95.25 0)
+      (effects (font (size 1.27 1.27)) hide)
+    )
