File: SCAN2000_breakout/scan2000_breakout.kicad_sch (KiCad schematic)
At the start: 114 parts, among them J1 Banana socket, J10 Banana socket, J11 Banana socket, J12 Banana socket, J13 Banana socket, J14 Banana socket, J15 Banana socket, J16 Banana socket, J17 Banana socket, J18 Banana socket, J19 Banana socket, J2 Banana socket, J20 Banana socket, J21 IDC-Header_2x13, J22 Conn_02x10_Odd_Even, J23 Conn_01x02_Pin, J24 Conn_01x02_Pin, J3 Banana socket, J4 Banana socket, J5 Banana socket, J6 Banana socket, J7 Banana socket, J8 Banana socket, J9 Banana socket, U1 TLP3558A, U10 TLP3558A, U11 TLP3558A, U12 TLP3558A, U13 TLP3558A, U14 TLP3558A, U15 TLP3558A, U16 TLP3558A, U17 TLP3558A, U18 TLP3558A, U19 TLP3558A, U2 TLP3558A, U20 TLP3558A, U21 TLP3558A, U22 TLP3558A, U23 TLP3558A, U24 TLP3558A, U25 TLP3558A, U26 TLP3558A, U27 TLP3558A, U28 TLP3558A, U29 TLP3558A, U3 TLP3558A, U30 TLP3558A, U31 TLP3558A, U32 TLP3558A, U33 TLP3558A, U34 TLP3558A, U35 TLP3558A, U36 TLP3558A, U37 TLP3558A, U38 TLP3558A, U39 TLP3558A, U4 TLP3558A, U40 TLP3558A, U41 TLP3558A, U42 TLP3558A, U43 TLP3558A, U44 TLP3558A, U5 TLP3558A, U6 TLP3558A, U7 TLP3558A, U8 TLP3558A, U9 TLP3558A

Commit message: Updates after fabrication
Parts:
- J21: MFN Würth -> Amphenol; PN 61202622121 -> 71922-126LF
- R1, R14: value 0.05 -> 0.1; PN LVK12R050DER -> LVK12R100CER
Other:
- note added: "Best is to use "long" version, as it will allow cable strains on the flat cable."
- note added: "LVK12R010CER = 10mOhm 0.5W, therefore: 7A max LVK12R050CER = 50mOhm 0.5W, therefore: 3A max LVK12R100CER = 100mOhm 0.5W, therefore: 2A max Lower resistance means lower accuracy at lower currents."
- note removed: "LVK12R050DER = 50mOhm 0.5W Therefore: 3A max"
Changed lines of the file:
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@@
     (stroke (width 0) (type default))
   )
-  (text "LVK12R050DER  = 50mOhm 0.5W\nTherefore: 3A max" (at 322.58 241.3 0)
+  (text "LVK12R010CER  = 10mOhm 0.5W, therefore: 7A max\nLVK12R050CER  = 50mOhm 0.5W, therefore: 3A max\nLVK12R100CER  = 100mOhm 0.5W, therefore: 2A max\n\nLower resistance means lower accuracy at lower currents."
+    (at 322.58 241.3 0)
+    (effects (font (size 1.27 1.27)) (justify left bottom))
+  )
+  (text "Best is to use \"long\" version, as it will allow cable strains on the flat cable."
+    (at 15.24 96.52 0)
     (effects (font (size 1.27 1.27)) (justify left bottom))
   )
@@
     (effects (font (size 1.27 1.27)) (justify left bottom))
   )
-  (text "LVK12R050DER  = 50mOhm 0.5W\nTherefore: 3A max" (at 87.63 243.84 0)
+  (text "LVK12R010CER  = 10mOhm 0.5W, therefore: 7A max\nLVK12R050CER  = 50mOhm 0.5W, therefore: 3A max\nLVK12R100CER  = 100mOhm 0.5W, therefore: 2A max\n\nLower resistance means lower accuracy at lower currents."
+    (at 87.63 243.84 0)
     (effects (font (size 1.27 1.27)) (justify left bottom))
   )
@@
       (effects (font (size 1.27 1.27)) (justify right bottom))
     )
-    (property "Value" "0.05" (at 81.788 242.5773 0)
+    (property "Value" "0.1" (at 81.788 242.5773 0)
       (effects (font (size 1.27 1.27)) (justify right bottom))
     )
@@
       (effects (font (size 1.27 1.27)) hide)
     )
-    (property "Datasheet" "~" (at 80.01 241.3 0)
+    (property "Datasheet" "https://www.mouser.fr/datasheet/2/303/res_lvk-3082595.pdf" (at 80.01 241.3 0)
       (effects (font (size 1.27 1.27)) hide)
     )
@@
       (effects (font (size 1.27 1.27)) hide)
     )
-    (property "PN" "LVK12R050DER" (at 80.01 241.3 0)
+    (property "PN" "LVK12R100CER" (at 80.01 241.3 0)
       (effects (font (size 1.27 1.27)) hide)
     )
@@
       (effects (font (size 1.27 1.27)) (justify right bottom))
     )
-    (property "Value" "0.05" (at 316.738 240.0373 0)
+    (property "Value" "0.1" (at 316.738 240.0373 0)
       (effects (font (size 1.27 1.27)) (justify right bottom))
     )
@@
       (effects (font (size 1.27 1.27)) hide)
     )
-    (property "Datasheet" "~" (at 314.96 238.76 0)
+    (property "Datasheet" "https://www.mouser.fr/datasheet/2/303/res_lvk-3082595.pdf" (at 314.96 238.76 0)
       (effects (font (size 1.27 1.27)) hide)
     )
@@
       (effects (font (size 1.27 1.27)) hide)
     )
-    (property "PN" "LVK12R050DER" (at 314.96 238.76 0)
+    (property "PN" "LVK12R100CER" (at 314.96 238.76 0)
       (effects (font (size 1.27 1.27)) hide)
     )
@@
       (effects (font (size 1.27 1.27)) hide)
     )
-    (property "Datasheet" "https://www.we-online.com/components/products/datasheet/6120xx22121.pdf" (at 55.88 52.07 0)
+    (property "Datasheet" "https://cdn.amphenol-cs.com/media/wysiwyg/files/documentation/datasheet/boardwiretoboard/bwb_quickie.pdf" (at 55.88 52.07 0)
       (effects (font (size 1.27 1.27)) hide)
     )
-    (property "MFN" "Würth" (at 55.88 52.07 0)
+    (property "MFN" "Amphenol" (at 55.88 52.07 0)
       (effects (font (size 1.27 1.27)) hide)
     )
-    (property "PN" "61202622121" (at 55.88 52.07 0)
+    (property "PN" "71922-126LF" (at 55.88 52.07 0)
       (effects (font (size 1.27 1.27)) hide)
     )
